Commit message: リンク色統一

File: double_jisaku6dof_arm.urdf (robot description, URDF)
Before this commit: robot double_jisaku6dof_arm, 18 links, 17 joints
Joints:
- joint shfted_base_joint: origin xyz=-1.0 -1.0 0 rpy=0 0 0 -> xyz=-1.5 0.0 0 rpy=0 0 0
- joint shifted_Base_joint: origin xyz=-0.03 -0.02 0 rpy=0 0 0 -> xyz=+0.03 +0.02 0 rpy=0 0 0
