Commit message: jisaku_6dof_arm: test for one robot urdf in moving frame

File: jisaku6dof_arm.urdf (robot description, URDF)
Before this commit: robot jisaku6def_arm, 9 links, 8 joints
Links:
- link Base: geometry collision box size=0.02 0.02 0.05; visual box size=0.02 0.02 0.05
- link link1: geometry collision box size=0.01 0.01 0.1; visual box size=0.01 0.01 0.1
- link link2: geometry collision box size=0.01 0.01 0.3; visual box size=0.01 0.01 0.3
- link link3: geometry collision box size=0.01 0.01 0.2; visual box size=0.01 0.01 0.2
- link link4: geometry collision box size=0.01 0.01 0.2; visual box size=0.01 0.01 0.2
- link link5: geometry collision box size=0.01 0.01 0.05; visual box size=0.01 0.01 0.05
- link link6: geometry collision box size=0.01 0.01 0.1; visual box size=0.01 0.01 0.1
Joints:
- joint hand_no_saki_joint: axis 0 0 1 -> (none); limit lower=-2.617 upper=2.617 effort=30 velocity=1.571 -> (none)

File: kaiten_gosa_double_arm.urdf (robot description, URDF)
Before this commit: robot double_jisaku6dof_arm, 18 links, 17 joints
Joints:
- joint shifted_Base_joint: origin xyz=0.0 0.0 0 rpy=0 0 0.0872665 -> xyz=0.0 0.0 0 rpy=0.52 0.52 0.0872665

Commit message: base_joint 削除

File: jisaku6dof_arm.urdf (robot description, URDF)
Before this commit: robot jisaku6dof_arm, 9 links, 8 joints
Links:
- removed link Base
- link base: mass None -> 1; geometry collision box size=0.02 0.02 0.05; visual box size=0.02 0.02 0.05
Joints:
- removed joint Base_joint
- joint joint1: parent Base -> base
